File: files/IMU Raspberry Pi Breakout RevB.sch (EAGLE design)
At the start: 13 parts, among them J1 PIN20X2, J2 ADIS1648X/49X/54X, J4 455-1750-1-ND, U1 ADM7172ACPZ-3.3-R7

Commit message: Updated design to include resistors that link SPI1 to SPI0. Improved silkscreen art.
Parts:
- added R1, R2, R3, R4: 0, SparkFun-Resistors:RESISTOR0603
Connections:
- removed net MISO: J1.21, J2.DOUT, J3.MISO
- removed net MOSI: J1.19, J2.DIN, J3.MOSI
- removed net N$2: J1.26, JP1.3, JP2.3
- removed net N$3: J1.24, JP1.1, JP2.1
- removed net SCLK: J1.23, J2.SCLK, J3.SCLK
- new net SPI0_CS0: J1.24, JP1.1
- new net SPI0_CS1: J1.26, JP1.3
- new net SPI0_MISO: J1.21, J2.DOUT, R2.2
- new net SPI0_MOSI: J1.19, J2.DIN, R3.2
- new net SPI0_SCLK: J1.23, J2.SCLK, R1.2
- new net SPI1_CS0: J1.18, JP2.3
- new net SPI1_CS1: J1.16, JP2.1
- new net SPI1_MISO: J1.22, J3.MISO, R2.1
- new net SPI1_MOSI: J1.37, J3.MOSI, R3.1
- new net SPI1_SCLK: J1.13, J3.SCLK, R1.1
- net !CS_1MM: now also R4.2
- net !CS_2MM: now also R4.1
Other:
- note added: "Install R1-R4 to link SPI0 and SPI1"
- moved on the sheet: JP1, JP2
